File: pcb/BBSensor.kicad_pcb (KiCad board)
At the start: 2 copper layers, 6 parts, among them J1 Earth, P1 Conn_WallPlug_Earth

Commit message: feat: Create Scheme
add Temperatures

Issue #1
Parts:
- added C201: 100n, Capacitor_THT:C_Disc_D3.4mm_W2.1mm_P2.50mm, F.Cu at (255.0, 148.3)
- added C301: 100n, Capacitor_THT:C_Disc_D3.4mm_W2.1mm_P2.50mm, F.Cu at (428.2, 136.2)
- added D101: RED, LED_THT:LED_D5.0mm, F.Cu at (309.7, 45.9)
- added D102: GREEN, LED_THT:LED_D5.0mm, F.Cu at (276.4, 71.7)
- added R101: 1k, Resistor_THT:R_Axial_DIN0411_L9.9mm_D3.6mm_P12.70mm_Horizontal, F.Cu at (309.2, 39.6)
- added R102: 1k, Resistor_THT:R_Axial_DIN0411_L9.9mm_D3.6mm_P12.70mm_Horizontal, F.Cu at (292.6, 49.9)
- added R103: 1k, Resistor_THT:R_Axial_DIN0411_L9.9mm_D3.6mm_P12.70mm_Horizontal, F.Cu at (275.9, 65.3)
- added R104: 1k, Resistor_THT:R_Axial_DIN0411_L9.9mm_D3.6mm_P12.70mm_Horizontal, F.Cu at (309.2, 34.4)
- added R105: 1k, Resistor_THT:R_Axial_DIN0411_L9.9mm_D3.6mm_P12.70mm_Horizontal, F.Cu at (275.9, 60.2)
- added R106: 2k2, Resistor_THT:R_Axial_DIN0411_L9.9mm_D3.6mm_P12.70mm_Horizontal, F.Cu at (275.9, 55.0)
- added R107: 2k2, Resistor_THT:R_Axial_DIN0411_L9.9mm_D3.6mm_P12.70mm_Horizontal, F.Cu at (275.9, 49.9)
- added R108: 2k2, Resistor_THT:R_Axial_DIN0411_L9.9mm_D3.6mm_P12.70mm_Horizontal, F.Cu at (292.6, 44.7)
- added R109: 2k2, Resistor_THT:R_Axial_DIN0411_L9.9mm_D3.6mm_P12.70mm_Horizontal, F.Cu at (275.9, 44.7)
- added R110: 2k2, Resistor_THT:R_Axial_DIN0411_L9.9mm_D3.6mm_P12.70mm_Horizontal, F.Cu at (292.6, 39.6)
- added R150: 140, Resistor_THT:R_Axial_DIN0411_L9.9mm_D3.6mm_P12.70mm_Horizontal, F.Cu at (275.9, 39.6)
- added R151: 140, Resistor_THT:R_Axial_DIN0411_L9.9mm_D3.6mm_P12.70mm_Horizontal, F.Cu at (292.6, 34.4)
- added R153: 2k2, Resistor_THT:R_Axial_DIN0411_L9.9mm_D3.6mm_P12.70mm_Horizontal, F.Cu at (275.9, 34.4)
- added R301: 220, Resistor_THT:R_Axial_DIN0411_L9.9mm_D3.6mm_P12.70mm_Horizontal, F.Cu at (445.2, 131.8)
- added R302: 2k, Resistor_THT:R_Axial_DIN0411_L9.9mm_D3.6mm_P12.70mm_Horizontal, F.Cu at (428.6, 131.8)
- added R4004: 2k2, Resistor_THT:R_Axial_DIN0411_L9.9mm_D3.6mm_P12.70mm_Horizontal, F.Cu at (412.2, 117.6)
- added R4005: 10k, Resistor_THT:R_Axial_DIN0411_L9.9mm_D3.6mm_P12.70mm_Horizontal, F.Cu at (443.1, 83.1)
- added R4006: 10k, Resistor_THT:R_Axial_DIN0411_L9.9mm_D3.6mm_P12.70mm_Horizontal, F.Cu at (426.5, 88.3)
- added R4007: 4k7, Resistor_THT:R_Axial_DIN0411_L9.9mm_D3.6mm_P12.70mm_Horizontal, F.Cu at (426.5, 93.4)
- added R4008: 200, Resistor_THT:R_Axial_DIN0411_L9.9mm_D3.6mm_P12.70mm_Horizontal, F.Cu at (412.2, 122.8)
- added R4010: 200, Resistor_THT:R_Axial_DIN0411_L9.9mm_D3.6mm_P12.70mm_Horizontal, F.Cu at (426.5, 98.6)
- added R4011: 2k, Resistor_THT:R_Axial_DIN0411_L9.9mm_D3.6mm_P12.70mm_Horizontal, F.Cu at (443.1, 88.3)
- added R4104: 2k2, Resistor_THT:R_Axial_DIN0411_L9.9mm_D3.6mm_P12.70mm_Horizontal, F.Cu at (426.5, 103.7)
- added R4105: 10k, Resistor_THT:R_Axial_DIN0411_L9.9mm_D3.6mm_P12.70mm_Horizontal, F.Cu at (428.9, 108.9)
- added R4106: 10k, Resistor_THT:R_Axial_DIN0411_L9.9mm_D3.6mm_P12.70mm_Horizontal, F.Cu at (443.1, 93.4)
- added R4107: 4k7, Resistor_THT:R_Axial_DIN0411_L9.9mm_D3.6mm_P12.70mm_Horizontal, F.Cu at (426.5, 83.1)
- added R4108: 200, Resistor_THT:R_Axial_DIN0411_L9.9mm_D3.6mm_P12.70mm_Horizontal, F.Cu at (443.1, 98.6)
- added R4110: 200, Resistor_THT:R_Axial_DIN0411_L9.9mm_D3.6mm_P12.70mm_Horizontal, F.Cu at (459.8, 83.1)
- added R4111: 2k, Resistor_THT:R_Axial_DIN0411_L9.9mm_D3.6mm_P12.70mm_Horizontal, F.Cu at (428.9, 114.0)
- added R4204: 2k2, Resistor_THT:R_Axial_DIN0411_L9.9mm_D3.6mm_P12.70mm_Horizontal, F.Cu at (257.9, 110.7)
- added R4205: 10k, Resistor_THT:R_Axial_DIN0411_L9.9mm_D3.6mm_P12.70mm_Horizontal, F.Cu at (257.9, 105.5)
- added R4206: 10k, Resistor_THT:R_Axial_DIN0411_L9.9mm_D3.6mm_P12.70mm_Horizontal, F.Cu at (243.7, 140.0)
- added R4207: 4k7, Resistor_THT:R_Axial_DIN0411_L9.9mm_D3.6mm_P12.70mm_Horizontal, F.Cu at (274.6, 105.5)
- added R4208: 200, Resistor_THT:R_Axial_DIN0411_L9.9mm_D3.6mm_P12.70mm_Horizontal, F.Cu at (291.2, 100.4)
- added R4210: 200, Resistor_THT:R_Axial_DIN0411_L9.9mm_D3.6mm_P12.70mm_Horizontal, F.Cu at (260.3, 131.3)
- added R4211: 2k, Resistor_THT:R_Axial_DIN0411_L9.9mm_D3.6mm_P12.70mm_Horizontal, F.Cu at (257.9, 115.8)
- added R4304: 2k2, Resistor_THT:R_Axial_DIN0411_L9.9mm_D3.6mm_P12.70mm_Horizontal, F.Cu at (274.6, 115.8)
- added R4305: 10k, Resistor_THT:R_Axial_DIN0411_L9.9mm_D3.6mm_P12.70mm_Horizontal, F.Cu at (274.6, 110.7)
- added R4306: 10k, Resistor_THT:R_Axial_DIN0411_L9.9mm_D3.6mm_P12.70mm_Horizontal, F.Cu at (260.3, 126.1)
- added R4307: 4k7, Resistor_THT:R_Axial_DIN0411_L9.9mm_D3.6mm_P12.70mm_Horizontal, F.Cu at (257.9, 121.0)
- added R4308: 200, Resistor_THT:R_Axial_DIN0411_L9.9mm_D3.6mm_P12.70mm_Horizontal, F.Cu at (257.9, 100.4)
- added R4310: 200, Resistor_THT:R_Axial_DIN0411_L9.9mm_D3.6mm_P12.70mm_Horizontal, F.Cu at (274.6, 100.4)
- added R4311: 2k, Resistor_THT:R_Axial_DIN0411_L9.9mm_D3.6mm_P12.70mm_Horizontal, F.Cu at (243.7, 134.9)
- added R4404: 2k2, Resistor_THT:R_Axial_DIN0411_L9.9mm_D3.6mm_P12.70mm_Horizontal, F.Cu at (372.8, 39.6)
- added R4405: 10k, Resistor_THT:R_Axial_DIN0411_L9.9mm_D3.6mm_P12.70mm_Horizontal, F.Cu at (375.2, 65.3)
- added R4406: 10k, Resistor_THT:R_Axial_DIN0411_L9.9mm_D3.6mm_P12.70mm_Horizontal, F.Cu at (406.1, 34.4)
- added R4407: 4k7, Resistor_THT:R_Axial_DIN0411_L9.9mm_D3.6mm_P12.70mm_Horizontal, F.Cu at (389.5, 49.9)
- added R4408: 200, Resistor_THT:R_Axial_DIN0411_L9.9mm_D3.6mm_P12.70mm_Horizontal, F.Cu at (389.5, 44.7)
- added R4410: 200, Resistor_THT:R_Axial_DIN0411_L9.9mm_D3.6mm_P12.70mm_Horizontal, F.Cu at (375.2, 60.2)
- added R4411: 2k, Resistor_THT:R_Axial_DIN0411_L9.9mm_D3.6mm_P12.70mm_Horizontal, F.Cu at (372.8, 55.0)
- added R4504: 2k2, Resistor_THT:R_Axial_DIN0411_L9.9mm_D3.6mm_P12.70mm_Horizontal, F.Cu at (372.8, 34.4)
- added R4505: 10k, Resistor_THT:R_Axial_DIN0411_L9.9mm_D3.6mm_P12.70mm_Horizontal, F.Cu at (372.8, 49.9)
- added R4506: 10k, Resistor_THT:R_Axial_DIN0411_L9.9mm_D3.6mm_P12.70mm_Horizontal, F.Cu at (389.5, 39.6)
- added R4507: 4k7, Resistor_THT:R_Axial_DIN0411_L9.9mm_D3.6mm_P12.70mm_Horizontal, F.Cu at (358.6, 74.1)
- added R4508: 200, Resistor_THT:R_Axial_DIN0411_L9.9mm_D3.6mm_P12.70mm_Horizontal, F.Cu at (372.8, 44.7)
- added R4510: 200, Resistor_THT:R_Axial_DIN0411_L9.9mm_D3.6mm_P12.70mm_Horizontal, F.Cu at (389.5, 34.4)
- added R4511: 2k, Resistor_THT:R_Axial_DIN0411_L9.9mm_D3.6mm_P12.70mm_Horizontal, F.Cu at (358.6, 68.9)
- added R4604: 2k2, Resistor_THT:R_Axial_DIN0411_L9.9mm_D3.6mm_P12.70mm_Horizontal, F.Cu at (327.9, 134.9)
- added R4605: 10k, Resistor_THT:R_Axial_DIN0411_L9.9mm_D3.6mm_P12.70mm_Horizontal, F.Cu at (344.6, 126.1)
- added R4606: 10k, Resistor_THT:R_Axial_DIN0411_L9.9mm_D3.6mm_P12.70mm_Horizontal, F.Cu at (342.2, 105.5)
- added R4607: 4k7, Resistor_THT:R_Axial_DIN0411_L9.9mm_D3.6mm_P12.70mm_Horizontal, F.Cu at (342.2, 110.7)
- added R4608: 200, Resistor_THT:R_Axial_DIN0411_L9.9mm_D3.6mm_P12.70mm_Horizontal, F.Cu at (327.9, 140.0)
- added R4610: 200, Resistor_THT:R_Axial_DIN0411_L9.9mm_D3.6mm_P12.70mm_Horizontal, F.Cu at (342.2, 115.8)
- added R4611: 2k, Resistor_THT:R_Axial_DIN0411_L9.9mm_D3.6mm_P12.70mm_Horizontal, F.Cu at (358.8, 105.5)
- added R4704: 2k2, Resistor_THT:R_Axial_DIN0411_L9.9mm_D3.6mm_P12.70mm_Horizontal, F.Cu at (358.8, 100.4)
- added R4705: 10k, Resistor_THT:R_Axial_DIN0411_L9.9mm_D3.6mm_P12.70mm_Horizontal, F.Cu at (342.2, 121.0)
- added R4706: 10k, Resistor_THT:R_Axial_DIN0411_L9.9mm_D3.6mm_P12.70mm_Horizontal, F.Cu at (358.8, 110.7)
- added R4707: 4k7, Resistor_THT:R_Axial_DIN0411_L9.9mm_D3.6mm_P12.70mm_Horizontal, F.Cu at (358.8, 115.8)
- added R4708: 200, Resistor_THT:R_Axial_DIN0411_L9.9mm_D3.6mm_P12.70mm_Horizontal, F.Cu at (375.5, 100.4)
- added R4710: 200, Resistor_THT:R_Axial_DIN0411_L9.9mm_D3.6mm_P12.70mm_Horizontal, F.Cu at (342.2, 100.4)
- added R4711: 2k, Resistor_THT:R_Axial_DIN0411_L9.9mm_D3.6mm_P12.70mm_Horizontal, F.Cu at (344.6, 131.3)
- added RV4001: 405, Potentiometer_THT:Potentiometer_Bourns_3296Y_Vertical, F.Cu at (435.0, 118.5)
- added RV4002: 300, Potentiometer_THT:Potentiometer_Bourns_3296Y_Vertical, F.Cu at (463.4, 112.3)
- added RV4009: 470, Potentiometer_THT:Potentiometer_Bourns_3296Y_Vertical, F.Cu at (463.4, 105.9)
- added RV4101: 405, Potentiometer_THT:Potentiometer_Bourns_3296Y_Vertical, F.Cu at (477.7, 94.3)
- added RV4102: 300, Potentiometer_THT:Potentiometer_Bourns_3296Y_Vertical, F.Cu at (465.9, 99.5)
- added RV4109: 470, Potentiometer_THT:Potentiometer_Bourns_3296Y_Vertical, F.Cu at (446.2, 118.5)
- added RV4201: 405, Potentiometer_THT:Potentiometer_Bourns_3296Y_Vertical, F.Cu at (294.9, 129.5)
- added RV4202: 300, Potentiometer_THT:Potentiometer_Bourns_3296Y_Vertical, F.Cu at (266.5, 135.8)
- added RV4209: 470, Potentiometer_THT:Potentiometer_Bourns_3296Y_Vertical, F.Cu at (277.6, 135.8)
- added RV4301: 405, Potentiometer_THT:Potentiometer_Bourns_3296Y_Vertical, F.Cu at (297.4, 116.7)
- added RV4302: 300, Potentiometer_THT:Potentiometer_Bourns_3296Y_Vertical, F.Cu at (309.1, 111.6)
- added RV4309: 470, Potentiometer_THT:Potentiometer_Bourns_3296Y_Vertical, F.Cu at (294.9, 123.1)
- added RV4401: 405, Potentiometer_THT:Potentiometer_Bourns_3296Y_Vertical, F.Cu at (409.8, 63.6)
- added RV4402: 300, Potentiometer_THT:Potentiometer_Bourns_3296Y_Vertical, F.Cu at (381.4, 69.8)
- added RV4409: 470, Potentiometer_THT:Potentiometer_Bourns_3296Y_Vertical, F.Cu at (409.8, 57.2)
- added RV4501: 405, Potentiometer_THT:Potentiometer_Bourns_3296Y_Vertical, F.Cu at (424.0, 45.6)
- added RV4502: 300, Potentiometer_THT:Potentiometer_Bourns_3296Y_Vertical, F.Cu at (412.3, 50.8)
- added RV4509: 470, Potentiometer_THT:Potentiometer_Bourns_3296Y_Vertical, F.Cu at (392.5, 69.8)
- added RV4601: 405, Potentiometer_THT:Potentiometer_Bourns_3296Y_Vertical, F.Cu at (379.1, 129.5)
- added RV4602: 300, Potentiometer_THT:Potentiometer_Bourns_3296Y_Vertical, F.Cu at (379.1, 123.1)
- added RV4609: 470, Potentiometer_THT:Potentiometer_Bourns_3296Y_Vertical, F.Cu at (393.4, 111.6)
- added RV4701: 405, Potentiometer_THT:Potentiometer_Bourns_3296Y_Vertical, F.Cu at (350.7, 135.8)
- added RV4702: 300, Potentiometer_THT:Potentiometer_Bourns_3296Y_Vertical, F.Cu at (361.9, 135.8)
- added RV4709: 470, Potentiometer_THT:Potentiometer_Bourns_3296Y_Vertical, F.Cu at (381.6, 116.7)
- added SW1: SW_Push, Button_Switch_THT:SW_Tactile_SPST_Angled_PTS645Vx83-2LFS, F.Cu at (293.6, 61.3)
- added TH1: Thermistor_NTC, Lumberg:LUMBERG_1553_02, F.Cu at (416.9, 86.2)
- added TH2: Thermistor_NTC, Lumberg:LUMBERG_1553_02, F.Cu at (416.9, 103.4)
- added TH3: Thermistor_NTC, Lumberg:LUMBERG_1553_02, F.Cu at (248.3, 103.4)
- added TH4: Thermistor_NTC, Lumberg:LUMBERG_1553_02, F.Cu at (248.3, 120.7)
- added TH5: Thermistor_NTC, Lumberg:LUMBERG_1553_02, F.Cu at (363.2, 37.5)
- added TH6: Thermistor_NTC, Lumberg:LUMBERG_1553_02, F.Cu at (363.2, 54.7)
- added TH7: Thermistor_NTC, Lumberg:LUMBERG_1553_02, F.Cu at (332.6, 120.7)
- added TH8: Thermistor_NTC, Lumberg:LUMBERG_1553_02, F.Cu at (332.6, 103.4)
- added U1: ESP8266-12E_NodeMCU_Lolin, Collection:ESP8266-12E_NodeMCU_Lolin, F.Cu at (257.8, 43.7)
- added U100: OPA2340, Package_DIP:DIP-8_W7.62mm_Socket, F.Cu at (459.9, 87.8)
- added U101: OPA2340, Package_DIP:DIP-8_W7.62mm_Socket, F.Cu at (445.6, 103.3)
- added U102: OPA2340, Package_DIP:DIP-8_W7.62mm_Socket, F.Cu at (308.0, 99.9)
- added U103: OPA2340, Package_DIP:DIP-8_W7.62mm_Socket, F.Cu at (277.1, 120.5)
- added U104: OPA2340, Package_DIP:DIP-8_W7.62mm_Socket, F.Cu at (392.0, 54.6)
- added U105: OPA2340, Package_DIP:DIP-8_W7.62mm_Socket, F.Cu at (406.2, 39.1)
- added U106: OPA2340, Package_DIP:DIP-8_W7.62mm_Socket, F.Cu at (375.6, 105.1)
- added U107: OPA2340, Package_DIP:DIP-8_W7.62mm_Socket, F.Cu at (361.3, 120.5)
- added U110: OPA2340, Package_DIP:DIP-8_W7.62mm_Socket, F.Cu at (476.5, 82.7)
- added U120: OPA2340, Package_DIP:DIP-8_W7.62mm_Socket, F.Cu at (291.3, 105.1)
- added U130: OPA2340, Package_DIP:DIP-8_W7.62mm_Socket, F.Cu at (422.9, 34.0)
- added U140: OPA2340, Package_DIP:DIP-8_W7.62mm_Socket, F.Cu at (392.2, 99.9)
- added U2: MCP3208, Package_DIP:DIP-16_W7.62mm_Socket, F.Cu at (243.8, 148.6)
- added U3: 74HC595, Package_DIP:DIP-16_W7.62mm_Socket, F.Cu at (416.9, 131.4)
- added U4: HD44780, Connector_PinSocket_2.54mm:PinSocket_1x16_P2.54mm_Vertical, F.Cu at (412.6, 131.6)
- D1: value LED -> POWER
- R1: value R -> 220; footprint Resistor_THT:R_Axial_DIN0414_L11.9mm_D4.5mm_P7.62mm_Vertical -> Resistor_THT:R_Axial_DIN0411_L9.9mm_D3.6mm_P12.70mm_Horizontal
Connections:
- PS1 pad 1: (no net) -> Net-(P1-Pad2)
- PS1 pad 2: Net-(F1-Pad2) -> Net-(P1-Pad1)
- PS1 pad 3: GND -> Net-(PS1-Pad3)
- PS1 pad 4: (no net) -> GND
- PS1 pad 5: Net-(P1-Pad1) -> Net-(F1-Pad2)

Commit message: feat: Create Scheme
switch 4-8 with normal sensors, add test PCB

Issue #1
Parts:
- removed R4404, R4504, R4604, R4704: 2k2, Resistor_THT:R_Axial_DIN0411_L9.9mm_D3.6mm_P12.70mm_Horizontal
- removed R4405, R4406, R4505, R4506, R4605, R4606, R4705, R4706: 10k, Resistor_THT:R_Axial_DIN0411_L9.9mm_D3.6mm_P12.70mm_Horizontal
- removed R4407, R4507, R4607, R4707: 4k7, Resistor_THT:R_Axial_DIN0411_L9.9mm_D3.6mm_P12.70mm_Horizontal
- removed R4408, R4410, R4508, R4510, R4608, R4610, R4708, R4710: 200, Resistor_THT:R_Axial_DIN0411_L9.9mm_D3.6mm_P12.70mm_Horizontal
- removed R4411, R4511, R4611, R4711: 2k, Resistor_THT:R_Axial_DIN0411_L9.9mm_D3.6mm_P12.70mm_Horizontal
- removed RV4401, RV4501, RV4601, RV4701: 405, Potentiometer_THT:Potentiometer_Bourns_3296Y_Vertical
- removed RV4402, RV4502, RV4602, RV4702: 300, Potentiometer_THT:Potentiometer_Bourns_3296Y_Vertical
- removed RV4409, RV4509, RV4609, RV4709: 470, Potentiometer_THT:Potentiometer_Bourns_3296Y_Vertical
- removed TH5, TH6, TH7, TH8: Thermistor_NTC, Lumberg:LUMBERG_1553_02
- removed U104, U105, U106, U107, U130, U140: OPA2340, Package_DIP:DIP-8_W7.62mm_Socket
- added C501: 100n, Capacitor_THT:C_Disc_D3.4mm_W2.1mm_P2.50mm, F.Cu at (128.9, 113.0)
- added C502: 100n, Capacitor_THT:C_Disc_D3.4mm_W2.1mm_P2.50mm, F.Cu at (141.0, 113.0)
- added C503: 100n, Capacitor_THT:C_Disc_D3.4mm_W2.1mm_P2.50mm, F.Cu at (153.0, 113.2)
- added C504: 100n, Capacitor_THT:C_Disc_D3.4mm_W2.1mm_P2.50mm, F.Cu at (165.1, 113.0)
- added J501: AudioJack2_SwitchT, Lumberg:LUMBERG_1501_09, F.Cu at (127.0, 141.9)
- added J502: AudioJack2_SwitchT, Lumberg:LUMBERG_1501_09, F.Cu at (136.5, 141.9)
- added J503: AudioJack2_SwitchT, Lumberg:LUMBERG_1501_09, F.Cu at (146.1, 141.9)
- added J504: AudioJack2_SwitchT, Lumberg:LUMBERG_1501_09, F.Cu at (155.6, 141.9)
- added R501: 10k, Resistor_THT:R_Axial_DIN0411_L9.9mm_D3.6mm_P12.70mm_Horizontal, F.Cu at (132.7, 113.0)
- added R502: 10k, Resistor_THT:R_Axial_DIN0411_L9.9mm_D3.6mm_P12.70mm_Horizontal, F.Cu at (144.8, 113.0)
- added R503: 10k, Resistor_THT:R_Axial_DIN0411_L9.9mm_D3.6mm_P12.70mm_Horizontal, F.Cu at (156.8, 113.2)
- added R504: 10k, Resistor_THT:R_Axial_DIN0411_L9.9mm_D3.6mm_P12.70mm_Horizontal, F.Cu at (168.9, 113.0)
- added RV501: 10k, Potentiometer_THT:Potentiometer_Bourns_3296Y_Vertical, F.Cu at (125.7, 117.5)
- added RV502: 10k, Potentiometer_THT:Potentiometer_Bourns_3296Y_Vertical, F.Cu at (137.8, 117.5)
- added RV503: 10k, Potentiometer_THT:Potentiometer_Bourns_3296Y_Vertical, F.Cu at (149.9, 117.5)
- added RV504: 10k, Potentiometer_THT:Potentiometer_Bourns_3296Y_Vertical, F.Cu at (161.9, 117.5)
- added ~: MountingHole_3.7mm_Pad, MountingHole:MountingHole_3.7mm_Pad, F.Cu at (37.0, 129.0)
- added ~: MountingHole_3.7mm_Pad, MountingHole:MountingHole_3.7mm_Pad, F.Cu at (177.0, 129.0)
- added ~: MountingHole_3.7mm_Pad, MountingHole:MountingHole_3.7mm_Pad, F.Cu at (177.0, 29.0)
- added ~: MountingHole_3.7mm_Pad, MountingHole:MountingHole_3.7mm_Pad, F.Cu at (37.0, 29.0)
- D1, D101, D102: footprint LED_THT:LED_D5.0mm -> VCC:5600F
- U4: footprint Connector_PinSocket_2.54mm:PinSocket_1x16_P2.54mm_Vertical -> Box_Header:Box_Header_Straight_2x08
- moved R301 398.4 mm to (48.3, 97.8), turned to 270 degrees
- moved C301 369.5 mm to (61.6, 90.2)
- moved U100 369.3 mm to (90.8, 99.8), turned to 90 degrees
- moved U3 364.9 mm to (54.0, 93.3)
- moved R302 362.6 mm to (66.7, 110.0)
- moved RV4102 360.1 mm to (108.0, 60.3)
- moved RV4002 356.6 mm to (108.0, 83.8)
- moved U101 355.9 mm to (90.8, 76.2), turned to 90 degrees
- moved RV4101 354.9 mm to (124.1, 62.9), turned to 180 degrees
- moved RV4009 350.3 mm to (113.7, 86.4), turned to 180 degrees
- moved TH1 347.6 mm to (73.0, 136.9), turned to 180 degrees
- moved U110 342.1 mm to (134.5, 87.9), turned to 90 degrees
- moved R4005 340.8 mm to (102.9, 102.2), turned to 90 degrees
- moved RV4109 337.1 mm to (113.7, 62.9), turned to 180 degrees
- moved R4106 336.9 mm to (107.3, 66.0), turned to 270 degrees
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Routing:
- net +5V: track 0.00 -> 719.7 mm
- net /Analog/Digital/TEMP5: track 0.00 -> 217.2 mm
- net /Analog/Digital/TEMP6: track 0.00 -> 204.7 mm
- net /Analog/Digital/TEMP7: track 0.00 -> 192.2 mm
- net Net-(TH4-Pad1): track 0.00 -> 181.6 mm
- net /Analog/Digital/TEMP8: track 0.00 -> 180.7 mm
- net Net-(R4304-Pad1): track 0.00 -> 178.6 mm
- net Net-(R4104-Pad1): track 0.00 -> 178.1 mm
- net /Analog/Digital/TEMP3: track 0.00 -> 166.0 mm, vias 0 -> 1
- net Net-(R4204-Pad1): track 0.00 -> 132.0 mm
- net /Analog/Digital/TEMP4: track 0.00 -> 128.3 mm
- net /Analog/Digital/TEMP1: track 0.00 -> 119.5 mm
- net Net-(TH2-Pad1): track 0.00 -> 118.6 mm
- net Net-(R4004-Pad1): track 0.00 -> 118.1 mm
- net Net-(R153-Pad1): track 0.00 -> 105.6 mm
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- added copper zone on B.Cu, net GND
Other:
- board outline added: 180 x 126 mm
- net class Default: trace_width 0.25 -> 0.3
- net class Large added: clearance 0.2, trace_width 4, via_dia 0.8, via_drill 0.4
- net class Medium added: clearance 0.2, trace_width 1, via_dia 0.8, via_drill 0.4
- rule pad_to_mask_clearance: 0 -> 0.051
- board text added: "BBSensor V1.0"
- board text added: "BOT"
- board text added: "TOP"
