File: pcb/BBSensor.kicad_pcb (KiCad board)
At the start: 2 copper layers, 180 x 126 mm, 118 parts, among them J1 Earth, J501 AudioJack2_SwitchT, J502 AudioJack2_SwitchT, J503 AudioJack2_SwitchT, J504 AudioJack2_SwitchT, P1 Conn_WallPlug_Earth, SW1 SW_Push, U1 ESP8266-12E_NodeMCU_Lolin, U100 OPA2340, U101 OPA2340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

Commit message: feat: Create Scheme
redo voltage amps for Pt100 with Testpoints

Issue #1
Parts:
- removed TP4002, TP4011, TP4102, TP4111, TP4202, TP4211, TP4302, TP4311: TestPoint, TestPoint:TestPoint_THTPad_D2.5mm_Drill1.2mm
- TP4001, TP4004, TP4009, TP4101, TP4104, TP4109, TP4201, TP4204, TP4209, TP4301, TP4304, TP4309, TP501, TP502, TP503, TP504: footprint TestPoint:TestPoint_THTPad_D2.5mm_Drill1.2mm -> TestPoint:TestPoint_Pad_D1.5mm
- moved TP4001 130.2 mm to (124.5, 91.4), turned to 180 degrees
- moved TP4009 125.4 mm to (124.5, 95.9), turned to 180 degrees
- moved TP4101 122.2 mm to (124.5, 76.8)
- moved TP4004 119.3 mm to (130.8, 91.4), turned to 180 degrees
- moved TP4109 114.9 mm to (124.5, 72.4)
- moved TP4104 111.4 mm to (130.8, 76.8)
- moved TP501 77.3 mm to (132.7, 109.2)
- moved TP1 73.5 mm to (163.8, 133.3)
- moved TP2 71.3 mm to (163.8, 139.1)
- moved TP502 65.5 mm to (144.8, 109.2)
- moved TP503 57.8 mm to (156.8, 109.2)
- moved TP4201 47.9 mm to (181.0, 91.4), turned to 180 degrees
- moved TP504 46.1 mm to (168.9, 109.2)
- moved TP4209 42.7 mm to (181.0, 95.9), turned to 180 degrees
- moved TP4301 42.0 mm to (181.0, 76.8)
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Routing:
- net GND: track 0.00 -> 792.3 mm
- net +5V: track 714.7 -> 660.6 mm
- net Net-(R4110-Pad2): track 48.7 -> 69.8 mm
- net Net-(R4010-Pad2): track 49.6 -> 70.6 mm
- net Net-(R4210-Pad2): track 49.5 -> 70.4 mm
- net Net-(R4310-Pad2): track 49.2 -> 69.9 mm
- net /Analog/Digital/SPI1: track 77.8 -> 57.8 mm
- net /Analog/Digital/TEMP4: track 128.3 -> 143.9 mm
- net /Analog/Digital/TEMP7: track 192.2 -> 207.7 mm
- net /Analog/Digital/TEMP8: track 180.7 -> 196.1 mm
- net Net-(TH1-Pad1): track 58.6 -> 73.8 mm
- net /Analog/Digital/TEMP6: track 204.7 -> 219.0 mm
- net /Analog/Digital/TEMP5: track 217.2 -> 230.5 mm
- net Net-(R4108-Pad2): track 47.4 -> 57.4 mm
- net Net-(R4008-Pad2): track 63.3 -> 73.2 mm
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Other:
- net class Medium: trace_width 1 -> 0.6
- board text added: "+5V"
- board text added: "GND"

Commit message: feat: Create PCB
Create and fix PCB

Issue #2
Parts:
- P1: footprint Bulgin:PF0030PC -> Bulgin:PX0580PC
- moved J1 24.2 mm to (176.5, 20.3)
- moved P1 15.6 mm to (147.3, 16.2), turned to 0 degrees
Routing:
- net Net-(P1-Pad1): track 44.9 -> 20.8 mm
- net Net-(P1-Pad2): track 26.4 -> 41.3 mm
- net Net-(J1-Pad1): track 32.2 -> 37.5 mm
- net /Analog/Digital/TEMP1: track 115.4 -> 114.2 mm
- net /Analog/Digital/TEMP2: track 89.9 -> 88.9 mm
- net /Analog/Digital/TEMP4: track 143.9 -> 143.3 mm
- net /Analog/Digital/TEMP3: track 172.1 -> 171.5 mm
- net /Analog/Digital/TEMP5: track 230.5 -> 229.9 mm
- net /Analog/Digital/TEMP6: track 219.0 -> 218.4 mm
- net /Analog/Digital/TEMP7: track 207.7 -> 207.1 mm
- net /Analog/Digital/TEMP8: track 196.1 -> 195.5 mm
Other:
- outline, holes or cut-outs redrawn
